File: Hardware/Schematic.sch (EAGLE design)
At the start: 105 parts, among them IC1 BQ25180YBGR_BQ25180YBGR, IC2 DRV2605YZFR, IC3 BMA423_BMA423, IC9 RT6160AWSC, J1 503480-2400, J2 TC2030-IDC_TC2030-IDC, J4 KH-TYPE-C-16P, Q1 20V/4.2A/52mΩ/1.4W, Q3 SI1308EDL-T1-GE3, U1 NRF52840_QF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

Commit message: Update Schematic.sch
Fixed the values of the following components:
- ANT1
- IC3
- IC1
- J2
Please let me know if there are any other incorrect values by opening another issue.
Fixes #4
Parts:
- ANT1: value 2450AT18B100E_2450AT18B100E -> 2450AT18B100E
- IC1: value BQ25180YBGR_BQ25180YBGR -> BQ25180YBGR
- IC3: value BMA423_BMA423 -> BMA423
- J2: value TC2030-IDC_TC2030-IDC -> TC2030-IDC
Changed lines of the file:
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@@
 </classes>
 <parts>
-<part name="IC1" library="InkTime_v5" library_urn="urn:adsk.wipprod:fs.file:vf.tUwrbmbJTRevvyDZ4HcNKA" deviceset="BQ25180YBGR_BQ25180YBGR" device=""/>
+<part name="IC1" library="InkTime_v5" library_urn="urn:adsk.wipprod:fs.file:vf.tUwrbmbJTRevvyDZ4HcNKA" deviceset="BQ25180YBGR_BQ25180YBGR" device="" value="BQ25180YBGR"/>
 <part name="GND1" library="InkTime_v5" library_urn="urn:adsk.wipprod:fs.file:vf.tUwrbmbJTRevvyDZ4HcNKA" deviceset="SUPPLY1_GND" device="">
 <attribute name="GND" value=""/>
@@
 <attribute name="GND" value=""/>
 </part>
-<part name="IC3" library="InkTime_v5" library_urn="urn:adsk.wipprod:fs.file:vf.tUwrbmbJTRevvyDZ4HcNKA" deviceset="BMA423_BMA423" device=""/>
+<part name="IC3" library="InkTime_v5" library_urn="urn:adsk.wipprod:fs.file:vf.tUwrbmbJTRevvyDZ4HcNKA" deviceset="BMA423_BMA423" device="" value="BMA423"/>
 <part name="GND10" library="InkTime_v5" library_urn="urn:adsk.wipprod:fs.file:vf.tUwrbmbJTRevvyDZ4HcNKA" deviceset="SUPPLY1_GND" device="">
 <attribute name="GND" value=""/>
@@
 <attribute name="GND" value=""/>
 </part>
-<part name="ANT1" library="InkTime_v5" library_urn="urn:adsk.wipprod:fs.file:vf.tUwrbmbJTRevvyDZ4HcNKA" deviceset="2450AT18B100E_2450AT18B100E" device="" value="2450AT18B100E_2450AT18B100E"/>
+<part name="ANT1" library="InkTime_v5" library_urn="urn:adsk.wipprod:fs.file:vf.tUwrbmbJTRevvyDZ4HcNKA" deviceset="2450AT18B100E_2450AT18B100E" device="" value="2450AT18B100E"/>
 <part name="GND23" library="InkTime_v5" library_urn="urn:adsk.wipprod:fs.file:vf.tUwrbmbJTRevvyDZ4HcNKA" deviceset="SUPPLY1_GND" device="">
 <attribute name="GND" value=""/>
@@
 <attribute name="GND" value=""/>
 </part>
-<part name="J2" library="InkTime_v5" library_urn="urn:adsk.wipprod:fs.file:vf.tUwrbmbJTRevvyDZ4HcNKA" deviceset="TC2030-IDC_TC2030-IDC" device="" value="TC2030-IDC_TC2030-IDC"/>
+<part name="J2" library="InkTime_v5" library_urn="urn:adsk.wipprod:fs.file:vf.tUwrbmbJTRevvyDZ4HcNKA" deviceset="TC2030-IDC_TC2030-IDC" device="" value="TC2030-IDC"/>
 <part name="GND30" library="InkTime_v5" library_urn="urn:adsk.wipprod:fs.file:vf.tUwrbmbJTRevvyDZ4HcNKA" deviceset="SUPPLY1_GND" device="">
 <attribute name="GND" value=""/>
