File: Hardware/Schematic.sch (EAGLE design)
At the start: 105 parts, among them IC1 BQ25180YBGR, IC2 DRV2605YZFR, IC3 BMA423, IC9 RT6160AWSC, J1 503480-2400, J2 TC2030-IDC, J4 KH-TYPE-C-16P, Q1 20V/4.2A/52mΩ/1.4W, Q3 SI1308EDL-T1-GE3, U1 NRF52840_QF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

Commit message: Display resistors and capacitor value
Displayed the values of resistors and capacitors so as to ensure a more readable schematic.
Fixes #7
Parts:
- R17, R18: RESISTANCE (none) -> 3k3
- R2, R3, R4: RESISTANCE (none) -> 0
- R9: RESISTANCE (none) -> 10k
- R_PWR_EPD: value ERA-1AEB3401C_CPF0201D7K68C1 -> 10k; RESISTANCE (none) -> 10K

Commit message: Revert "Display resistors and capacitor value"
This reverts commit e3d6df2a964783730cc62ca4a1df47b7156c4929.
Parts:
- R17, R18: RESISTANCE 3k3 -> (none)
- R2, R3, R4: RESISTANCE 0 -> (none)
- R9: RESISTANCE 10k -> (none)
- R_PWR_EPD: value 10k -> ERA-1AEB3401C_CPF0201D7K68C1; RESISTANCE 10K -> (none)
